File: Logique/Carte OlINPiades 2017 - Logique.sch (KiCad schematic (older format))
At the start: 90 parts, among them P1 CONN_01X32, P2 CONN_01X32, P3 CONN_01X02, P4 CONN_01X06, P5 CONN_01X04, P6 CONN_01X02, P7 CONN_FREE_01X03, Q1 MMPQ2907A, Q2 MMPQ2907A, Q3 MMPQ2907A, Q4 MMPQ2907A, Q5 MMPQ2907A, Q6 MMPQ2907A, Q7 MMPQ2907A, Q8 MMPQ2907A, Q9 DSS4160T, U1 74AHC1G, U2 CD74HC154, U3 CD74HC154, U4 STM32F303K8, U5 NCP59301DSS33R4G, Y1 Crystal

Commit message: Kicad 5, argh !
Parts:
- C1, C2, C3, C4, C5, C6, C7, C8, C9: symbol C -> Device:C
- D17: symbol D -> Device:D
- JP1: symbol JUMPER3 -> Device:Jumper_NC_Dual
- JP2: symbol JUMPER -> Device:Jumper
- Q9: symbol Q_NPN_BEC -> Device:Q_NPN_BEC
- R1, R10, R11, R12, R13, R14, R15, R16, R17, R18, R19, R2, R20, R21, R22, R23, R24, R25, R26, R27, R28, R29, R3, R30, R31, R32, R33, R34, R35, R36, R37, R38, R4, R5, R6, R7, R8, R9: symbol R -> Device:R
- U4: symbol STM32F303K8 -> MCU_ST_STM32F3:STM32F303K8Tx
- Y1: symbol Crystal -> Device:Crystal
Connections:
- wire segments 468 -> 544

Commit message: Update schematics and PCB to kicad5
Parts:
- removed unit 1 of D1
- removed unit 1 of D10
- removed unit 1 of D11
- removed unit 1 of D12
- removed unit 1 of D13
- removed unit 1 of D14
- removed unit 1 of D15
- removed unit 1 of D16
- removed unit 1 of D2
- removed unit 1 of D3
- removed unit 1 of D4
- removed unit 1 of D5
- removed unit 1 of D6
- removed unit 1 of D7
- removed unit 1 of D8
- removed unit 1 of D9
- removed unit 2 of Q1
- removed unit 3 of Q1
- removed unit 4 of Q1
- removed Q2, Q3, Q4, Q5, Q6, Q7, Q8: MMPQ2907A, Housings_SOIC:SOIC-16_3.9x9.9mm_Pitch1.27mm, symbol MMPQ2907A
- added unit 2 of Q1
- added unit 3 of Q1
- added unit 4 of Q1
- added Q2, Q3, Q4, Q5, Q6, Q7, Q8: MMPQ2907A, Package_SO:SOIC-16_3.9x9.9mm_P1.27mm, symbol olinpiades:MMPQ2907
- C1, C2, C3, C4, C5, C7, C8: footprint Capacitors_SMD:C_0805_HandSoldering -> Capacitor_SMD:C_0805_2012Metric_Pad1.15x1.40mm_HandSolder
- C6, C9: footprint Capacitors_SMD:C_1206_HandSoldering -> Capacitor_SMD:C_1206_3216Metric_Pad1.42x1.75mm_HandSolder
- D1, D10, D11, D12, D13, D14, D15, D16, D2, D3, D4, D5, D6, D7, D8, D9: footprint TO_SOT_Packages_SMD:SOT-323 -> Package_TO_SOT_SMD:SOT-323_SC-70_Handsoldering; symbol BAT54CW -> Diode:BAT54CW
- D17: footprint Diodes_SMD:SMA_Handsoldering -> Diode_SMD:D_SMA_Handsoldering
- JP1: footprint Pin_Headers:Pin_Header_Straight_1x03_Pitch2.54mm -> Connector_PinHeader_2.54mm:PinHeader_1x03_P2.54mm_Vertical
- JP2, R37, R38: footprint Resistors_SMD:R_1206_HandSoldering -> Resistor_SMD:R_1206_3216Metric_Pad1.42x1.75mm_HandSolder
- P1, P2: footprint Pin_Headers:Pin_Header_Straight_1x32 -> Connector_PinHeader_2.54mm:PinHeader_1x32_P2.54mm_Vertical; symbol CONN_01X32 -> Connector_Generic:Conn_01x32
- P3, P6: footprint Connectors_Molex_Complete:Molex_MiniFit-JR-5556-02A_2x01x4.20mm_Straight -> Connector_Molex:Molex_Mini-Fit_Jr_5566-02A_2x01_P4.20mm_Vertical; symbol CONN_01X02 -> Connector_Generic:Conn_01x02
- P4: footprint Pin_Headers:Pin_Header_Angled_1x06_Pitch2.54mm -> Connector_PinHeader_2.54mm:PinHeader_1x06_P2.54mm_Horizontal; symbol CONN_01X06 -> Connector_Generic:Conn_01x06
- P5: footprint Pin_Headers:Pin_Header_Angled_1x04_Pitch2.54mm -> Connector_PinHeader_2.54mm:PinHeader_1x04_P2.54mm_Horizontal; symbol CONN_01X04 -> Connector_Generic:Conn_01x04
- P7: footprint Pin_Headers:Pin_Header_Straight_1x03_Pitch2.54mm -> Connector_PinHeader_2.54mm:PinHeader_1x03_P2.54mm_Vertical; symbol CONN_01X03 -> Connector_Generic:Conn_01x03
- Q1: footprint Housings_SOIC:SOIC-16_3.9x9.9mm_Pitch1.27mm -> Package_SO:SOIC-16_3.9x9.9mm_P1.27mm; symbol MMPQ2907A -> olinpiades:MMPQ2907
- Q9: footprint TO_SOT_Packages_SMD:SOT-23_Handsoldering -> Package_TO_SOT_SMD:SOT-23_Handsoldering
- R1, R10, R11, R12, R13, R14, R15, R16, R17, R18, R19, R2, R20, R21, R22, R23, R24, R25, R26, R27, R28, R29, R3, R30, R31, R32, R34, R35, R36, R4, R5, R6, R7, R8, R9: footprint Resistors_SMD:R_0603_HandSoldering -> Resistor_SMD:R_0603_1608Metric_Pad1.05x0.95mm_HandSolder
- R33: footprint misc:SM_3 -> Resistor_SMD:R_4020_10251Metric_Pad1.65x5.30mm_HandSolder
- S1, S2: footprint Housings_SSOP:TSSOP-24_4.4x7.8mm_Pitch0.65mm -> Package_SO:TSSOP-24_4.4x7.8mm_P0.65mm; symbol CAT4016 -> olinpiades:CAT4016
- U1: footprint misc:SOT-23-5 -> Package_TO_SOT_SMD:SOT-23-5_HandSoldering; symbol 74AHC1G -> 74xGxx:74AHC1G04
- U2, U3: footprint Housings_SOIC:SOIC-24_7.5x15.4mm_Pitch1.27mm -> Package_SO:SOIC-24W_7.5x15.4mm_P1.27mm; symbol CD74HC154 -> olinpiades:CD74HC154
- U4: footprint Housings_QFP:LQFP-32_7x7mm_Pitch0.8mm -> Package_QFP:LQFP-32_7x7mm_P0.8mm
- U5: footprint TO_SOT_Packages_SMD:TO-263-5Lead -> Package_TO_SOT_SMD:TO-263-5_TabPin3; symbol NCP59301DSS33R4G -> olinpiades:NCP59301
- Y1: footprint Crystals:Crystal_HC49-4H_Vertical -> Crystal:Crystal_HC49-4H_Vertical
Connections:
- wire segments 544 -> 473
Other:
- note added: "Attention, vérifier la footprint\npar rapport au composant réel !! (R33)\n"
- moved on the sheet: C1, C2, R33, R34, R36
